File: hardware/ir_receiver/piLaz0rTag_receiver.kicad_pcb (KiCad board)
At the start: 2 copper layers, 30 x 30 mm, 4 parts

Commit message: Some rework on the receiver pcb
Parts:
- moved LED1 2.06 mm to (108.5, 94.0)
- moved Output1 1.50 mm to (114.5, 80.0)
Routing:
- net +5V: track 62.2 -> 58.2 mm
- net /LED_DOUT: track 9.42 -> 7.59 mm
- net /IR_DATA: track 22.7 -> 21.0 mm
- net /LED_DIN: track 9.80 -> 8.47 mm
Changed lines of the file:
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@@
     (links 12)
     (no_connects 0)
-    (area 89.924999 69.924999 120.075001 100.075001)
+    (area 88.666667 66.8 120.075001 100.075001)
     (thickness 1.6)
-    (drawings 4)
-    (tracks 19)
+    (drawings 6)
+    (tracks 23)
     (zones 0)
     (modules 4)
@@
   (page A4)
   (layers
-    (0 F.Cu signal)
+    (0 F.Cu signal hide)
     (31 B.Cu signal)
     (32 B.Adhes user)
@@
   )
   (module Socket_Strips:Socket_Strip_Straight_1x05_Pitch2.54mm (layer F.Cu)
-    (at 94 80)
+    (at 114.5 80)
     (descr "Through hole straight socket strip, 1x05, 2.54mm pitch, single row")
     (tags "Through hole socket strip THT 1x05 2.54mm single row")
-    (fp_text reference Input1 (at 0 -2.33) (layer F.SilkS)
+    (fp_text reference Output1 (at 0 -2.33) (layer F.SilkS)
       (effects (font (size 1 1) (thickness 0.15)))
     )
@@
       (net 3 /IR_DATA))
     (pad 5 thru_hole circle (at 0 10.16) (size 2 2) (drill 0.8) (layers *.Cu *.Mask)
-      (net 4 /LED_DIN))
+      (net 5 /LED_DOUT))
     (model ${KISYS3DMOD}/Socket_Strips.3dshapes/Socket_Strip_Straight_1x05_Pitch2.54mm.wrl
       (at (xyz 0 -0.2 0))
@@
   )
   (module Socket_Strips:Socket_Strip_Straight_1x05_Pitch2.54mm (layer F.Cu)
-    (at 116 80)
+    (at 94 80)
     (descr "Through hole straight socket strip, 1x05, 2.54mm pitch, single row")
     (tags "Through hole socket strip THT 1x05 2.54mm single row")
-    (fp_text reference Output1 (at 0 -2.33) (layer F.SilkS)
+    (fp_text reference Input1 (at 0 -2.33) (layer F.SilkS)
       (effects (font (size 1 1) (thickness 0.15)))
     )
@@
       (net 3 /IR_DATA))
     (pad 5 thru_hole circle (at 0 10.16) (size 2 2) (drill 0.8) (layers *.Cu *.Mask)
-      (net 5 /LED_DOUT))
+      (net 4 /LED_DIN))
     (model ${KISYS3DMOD}/Socket_Strips.3dshapes/Socket_Strip_Straight_1x05_Pitch2.54mm.wrl
       (at (xyz 0 -0.2 0))
@@
   )
   (module Socket_Strips:Socket_Strip_Straight_1x04_Pitch2.54mm (layer F.Cu)
-    (at 109 96 270)
+    (at 108.5 94 270)
     (descr "Through hole straight socket strip, 1x04, 2.54mm pitch, single row")
     (tags "Through hole socket strip THT 1x04 2.54mm single row")
@@
       (net 1 +5V))
   )
+  (dimension 30 (width 0.3) (layer Eco2.User)
+    (gr_text "30,000 mm" (at 122 85 90) (layer Eco2.User)
+      (effects (font (size 1.5 1.5) (thickness 0.3)))
+    )
+    (feature1 (pts (xy 122 70) (xy 122 70)))
+    (feature2 (pts (xy 122 100) (xy 122 100)))
+    (crossbar (pts (xy 122 100) (xy 122 70)))
+    (arrow1a (pts (xy 122 70) (xy 122.586421 71.126504)))
+    (arrow1b (pts (xy 122 70) (xy 121.413579 71.126504)))
+    (arrow2a (pts (xy 122 100) (xy 122.586421 98.873496)))
+    (arrow2b (pts (xy 122 100) (xy 121.413579 98.873496)))
+  )
+  (dimension 30 (width 0.3) (layer Eco2.User)
+    (gr_text "30,000 mm" (at 105 68) (layer Eco2.User)
+      (effects (font (size 1.5 1.5) (thickness 0.3)))
+    )
+    (feature1 (pts (xy 120 68) (xy 120 68)))
+    (feature2 (pts (xy 90 68) (xy 90 68)))
+    (crossbar (pts (xy 90 68) (xy 120 68)))
+    (arrow1a (pts (xy 120 68) (xy 118.873496 68.586421)))
+    (arrow1b (pts (xy 120 68) (xy 118.873496 67.413579)))
+    (arrow2a (pts (xy 90 68) (xy 91.126504 68.586421)))
+    (arrow2b (pts (xy 90 68) (xy 91.126504 67.413579)))
+  )
   (gr_line (start 120 100) (end 90 100) (angle 90) (layer Edge.Cuts) (width 0.15))
   (gr_line (start 120 70) (end 120 100) (angle 90) (layer Edge.Cuts) (width 0.15))
   (gr_line (start 90 70) (end 120 70) (angle 90) (layer Edge.Cuts) (width 0.15))
   (gr_line (start 90 100) (end 90 70) (angle 90) (layer Edge.Cuts) (width 0.15))
-  (segment (start 109.4 82.32) (end 109.48 82.32) (width 1) (layer B.Cu) (net 1) (status C00000))
-  (segment (start 109.48 82.32) (end 111.8 80) (width 1) (layer B.Cu) (net 1) (status 400000))
-  (segment (start 111.8 80) (end 116 80) (width 1) (layer B.Cu) (net 1) (status 800000))
-  (segment (start 94 80) (end 107.08 80) (width 1) (layer B.Cu) (net 1) (status 400000))
-  (segment (start 107.08 80) (end 109.4 82.32) (width 1) (layer B.Cu) (net 1) (status 800000))
-  (segment (start 119 99) (end 119 83) (width 1) (layer B.Cu) (net 1))
-  (segment (start 103.92 98.92) (end 104 99) (width 1) (layer B.Cu) (net 1))
-  (segment (start 104 99) (end 119 99) (width 1) (layer B.Cu) (net 1))
-  (segment (start 103.92 96) (end 103.92 98.92) (width 1) (layer B.Cu) (net 1))
-  (segment (start 119 83) (end 116 80) (width 1) (layer B.Cu) (net 1))
-  (segment (start 109.4 87.4) (end 94.22 87.4) (width 1) (layer B.Cu) (net 3) (status C00000))
-  (segment (start 94.22 87.4) (end 94 87.62) (width 1) (layer B.Cu) (net 3) (status C00000))
-  (segment (start 109.4 87.4) (end 115.78 87.4) (width 1) (layer B.Cu) (net 3) (status C00000))
-  (segment (start 115.78 87.4) (end 116 87.62) (width 1) (layer B.Cu) (net 3) (status C00000))
-  (segment (start 115.62 88) (end 116 87.62) (width 0.25) (layer B.Cu) (net 3))
-  (segment (start 94 90.16) (end 95.54 90.16) (width 1) (layer B.Cu) (net 4))
-  (segment (start 95.54 90.16) (end 101.38 96) (width 1) (layer B.Cu) (net 4))
-  (segment (start 109 96) (end 110.16 96) (width 1) (layer B.Cu) (net 5))
-  (segment (start 110.16 96) (end 116 90.16) (width 1) (layer B.Cu) (net 5))
+  (segment (start 114.5 80) (end 117 80) (width 1) (layer B.Cu) (net 1))
+  (segment (start 103.42 96.42) (end 103.42 94) (width 1) (layer B.Cu) (net 1))
+  (segment (start 104.5 97.5) (end 103.42 96.42) (width 1) (layer B.Cu) (net 1))
+  (segment (start 113.5 97.5) (end 104.5 97.5) (width 1) (layer B.Cu) (net 1))
+  (segment (start 117.5 93.5) (end 113.5 97.5) (width 1) (layer B.Cu) (net 1))
+  (segment (start 117.5 80.5) (end 117.5 93.5) (width 1) (layer B.Cu) (net 1))
+  (segment (start 117 80) (end 117.5 80.5) (width 1) (layer B.Cu) (net 1))
+  (segment (start 109.4 82.32) (end 109.4 82.1) (width 1) (layer B.Cu) (net 1))
+  (segment (start 109.4 82.1) (end 111.5 80) (width 1) (layer B.Cu) (net 1))
+  (segment (start 111.5 80) (end 114.5 80) (width 1) (layer B.Cu) (net 1))
+  (segment (start 109.4 82.32) (end 109.4 81.6) (width 1) (layer B.Cu) (net 1))
+  (segment (start 109.4 82.32) (end 109.48 82.32) (width 1) (layer B.Cu) (net 1))
+  (segment (start 94 80) (end 107.08 80) (width 1) (layer B.Cu) (net 1))
+  (segment (start 107.08 80) (end 109.4 82.32) (width 1) (layer B.Cu) (net 1))
+  (segment (start 109.4 87.4) (end 114.28 87.4) (width 1) (layer B.Cu) (net 3) (status C00000))
+  (segment (start 114.28 87.4) (end 114.5 87.62) (width 1) (layer B.Cu) (net 3) (status C00000))
+  (segment (start 114.28 87.4) (end 114.5 87.62) (width 1) (layer B.Cu) (net 3))
+  (segment (start 109.4 87.4) (end 94.22 87.4) (width 1) (layer B.Cu) (net 3))
+  (segment (start 94.22 87.4) (end 94 87.62) (width 1) (layer B.Cu) (net 3))
+  (segment (start 94 90.16) (end 97.04 90.16) (width 1) (layer B.Cu) (net 4))
+  (segment (start 97.04 90.16) (end 100.88 94) (width 1) (layer B.Cu) (net 4))
+  (segment (start 108.5 94) (end 110.66 94) (width 1) (layer B.Cu) (net 5))
+  (segment (start 110.66 94) (end 114.5 90.16) (width 1) (layer B.Cu) (net 5))
   (zone (net 2) (net_name GND) (layer B.Cu) (hatch edge 0.508)
     (connect_pads yes (clearance 0.6))

Commit message: Some rework on the receiver pcb
Parts:
- IR_REC1, Input1, LED1, Output1: moved to B.Cu
- moved Input1 23.5 mm to (94.0, 103.5)
- moved Output1 23.5 mm to (114.5, 103.5)
- moved IR_REC1 8.70 mm to (109.4, 96.1), turned to 270 degrees
- moved LED1 4.50 mm to (108.5, 89.5), turned to 90 degrees
Routing:
- added copper zone on F.Cu, net GND
- removed copper zone on B.Cu, net GND
