File: hardware/ir_receiver/piLaz0rTag_receiver.sch (KiCad schematic (older format))
At the start: 5 parts

Commit message: Make GND also in schemantic
Changed lines of the file:
@@
 $EndComp
 $Comp
-L GND #PWR10
+L GND #PWR01
 U 1 1 590CA8D5
 P 7150 2450
-F 0 "#PWR10" H 7150 2200 50  0001 C CNN
+F 0 "#PWR01" H 7150 2200 50  0001 C CNN
 F 1 "GND" H 7150 2300 50  0000 C CNN
 F 2 "" H 7150 2450 50  0001 C CNN
@@
 $EndComp
 $Comp
-L GND #PWR4
+L GND #PWR02
 U 1 1 590CA905
 P 4700 1350
-F 0 "#PWR4" H 4700 1100 50  0001 C CNN
+F 0 "#PWR02" H 4700 1100 50  0001 C CNN
 F 1 "GND" H 4700 1200 50  0000 C CNN
 F 2 "" H 4700 1350 50  0001 C CNN
@@
 $EndComp
 $Comp
-L +5V #PWR3
+L +5V #PWR03
 U 1 1 590CAA44
 P 3700 950
-F 0 "#PWR3" H 3700 800 50  0001 C CNN
+F 0 "#PWR03" H 3700 800 50  0001 C CNN
 F 1 "+5V" H 3700 1090 50  0000 C CNN
 F 2 "" H 3700 950 50  0001 C CNN
@@
 $EndComp
 $Comp
-L +5V #PWR9
+L +5V #PWR04
 U 1 1 590CAAB3
 P 6950 2450
-F 0 "#PWR9" H 6950 2300 50  0001 C CNN
+F 0 "#PWR04" H 6950 2300 50  0001 C CNN
 F 1 "+5V" H 6950 2590 50  0000 C CNN
 F 2 "" H 6950 2450 50  0001 C CNN
@@
 $EndComp
 $Comp
-L +5V #PWR5
+L +5V #PWR05
 U 1 1 5AF82ADB
 P 5400 2900
-F 0 "#PWR5" H 5400 2750 50  0001 C CNN
+F 0 "#PWR05" H 5400 2750 50  0001 C CNN
 F 1 "+5V" H 5400 3040 50  0000 C CNN
 F 2 "" H 5400 2900 50  0001 C CNN
@@
 $EndComp
 $Comp
-L +5V #PWR11
+L +5V #PWR06
 U 1 1 5AF82AFB
 P 7550 2900
-F 0 "#PWR11" H 7550 2750 50  0001 C CNN
+F 0 "#PWR06" H 7550 2750 50  0001 C CNN
 F 1 "+5V" H 7550 3040 50  0000 C CNN
 F 2 "" H 7550 2900 50  0001 C CNN
@@
 	-1   0    0    1
 $EndComp
-$Comp
-L GND #PWR6
-U 1 1 5AF82B3B
-P 5700 2900
-F 0 "#PWR6" H 5700 2650 50  0001 C CNN
-F 1 "GND" H 5700 2750 50  0000 C CNN
-F 2 "" H 5700 2900 50  0001 C CNN
-F 3 "" H 5700 2900 50  0001 C CNN
-	1    5700 2900
-	1    0    0    -1
-$EndComp
-Wire Wire Line
-	5900 2900 5900 3550
-Wire Wire Line
-	8050 3550 8050 2900
-Wire Wire Line
-	6100 2900 6650 2900
-Wire Wire Line
-	6650 2900 6650 950
-Wire Wire Line
-	6650 950  4700 950
 Text Label 6200 2900 0    60   ~ 0
 LedIn
-Wire Wire Line
-	3700 1350 3700 3700
-Wire Wire Line
-	3700 3700 8250 3700
-Wire Wire Line
-	8250 3700 8250 2900
 Text Label 4700 3700 0    60   ~ 0
 LedOut
-Wire Wire Line
-	7050 2450 7050 3550
-Connection ~ 7050 3550
 Text Label 6100 3550 0    60   ~ 0
 IrData
-$Comp
-L GND #PWR12
-U 1 1 5AF82E31
-P 7850 2900
-F 0 "#PWR12" H 7850 2650 50  0001 C CNN
-F 1 "GND" H 7850 2750 50  0000 C CNN
-F 2 "" H 7850 2900 50  0001 C CNN
-F 3 "" H 7850 2900 50  0001 C CNN
-	1    7850 2900
-	1    0    0    -1
-$EndComp
-Connection ~ 5900 3550
-Wire Wire Line
-	5900 3550 8050 3550
 $Comp
 L CP VStab1
@@
 $EndComp
 $Comp
-L +5V #PWR1
+L +5V #PWR07
 U 1 1 5AF9301E
 P 2900 2700
-F 0 "#PWR1" H 2900 2550 50  0001 C CNN
+F 0 "#PWR07" H 2900 2550 50  0001 C CNN
 F 1 "+5V" H 2900 2840 50  0000 C CNN
 F 2 "" H 2900 2700 50  0001 C CNN
@@
 $EndComp
 $Comp
-L GND #PWR2
+L GND #PWR08
 U 1 1 5AF9303C
 P 2900 3000
-F 0 "#PWR2" H 2900 2750 50  0001 C CNN
+F 0 "#PWR08" H 2900 2750 50  0001 C CNN
 F 1 "GND" H 2900 2850 50  0000 C CNN
 F 2 "" H 2900 3000 50  0001 C CNN
@@
 $EndComp
 $Comp
-L GND #PWR?
+L GND #PWR09
 U 1 1 5AFEA6A2
 P 5500 2900
-F 0 "#PWR?" H 5500 2650 50  0001 C CNN
+F 0 "#PWR09" H 5500 2650 50  0001 C CNN
 F 1 "GND" H 5500 2750 50  0000 C CNN
 F 2 "" H 5500 2900 50  0001 C CNN
@@
 $EndComp
 $Comp
-L GND #PWR?
+L GND #PWR010
 U 1 1 5AFEA6C0
 P 5600 2900
-F 0 "#PWR?" H 5600 2650 50  0001 C CNN
+F 0 "#PWR010" H 5600 2650 50  0001 C CNN
 F 1 "GND" H 5600 2750 50  0000 C CNN
 F 2 "" H 5600 2900 50  0001 C CNN
@@
 $EndComp
 $Comp
-L GND #PWR?
+L GND #PWR011
 U 1 1 5AFEA6DE
 P 5800 2900
-F 0 "#PWR?" H 5800 2650 50  0001 C CNN
+F 0 "#PWR011" H 5800 2650 50  0001 C CNN
 F 1 "GND" H 5800 2750 50  0000 C CNN
 F 2 "" H 5800 2900 50  0001 C CNN
@@
 $EndComp
 $Comp
-L GND #PWR?
+L GND #PWR012
 U 1 1 5AFEA6FC
 P 6000 2900
-F 0 "#PWR?" H 6000 2650 50  0001 C CNN
+F 0 "#PWR012" H 6000 2650 50  0001 C CNN
 F 1 "GND" H 6000 2750 50  0000 C CNN
 F 2 "" H 6000 2900 50  0001 C CNN
@@
 $EndComp
 $Comp
-L GND #PWR?
+L GND #PWR013
 U 1 1 5AFEA740
 P 7650 2900
-F 0 "#PWR?" H 7650 2650 50  0001 C CNN
+F 0 "#PWR013" H 7650 2650 50  0001 C CNN
 F 1 "GND" H 7650 2750 50  0000 C CNN
 F 2 "" H 7650 2900 50  0001 C CNN
@@
 $EndComp
 $Comp
-L GND #PWR?
+L GND #PWR014
 U 1 1 5AFEA75E
 P 7750 2900
-F 0 "#PWR?" H 7750 2650 50  0001 C CNN
+F 0 "#PWR014" H 7750 2650 50  0001 C CNN
 F 1 "GND" H 7750 2750 50  0000 C CNN
 F 2 "" H 7750 2900 50  0001 C CNN
@@
 $EndComp
 $Comp
-L GND #PWR?
+L GND #PWR015
 U 1 1 5AFEA77C
 P 7950 2900
-F 0 "#PWR?" H 7950 2650 50  0001 C CNN
+F 0 "#PWR015" H 7950 2650 50  0001 C CNN
 F 1 "GND" H 7950 2750 50  0000 C CNN
 F 2 "" H 7950 2900 50  0001 C CNN
@@
 $EndComp
 $Comp
-L GND #PWR?
+L GND #PWR016
 U 1 1 5AFEA79A
 P 8150 2900
-F 0 "#PWR?" H 8150 2650 50  0001 C CNN
+F 0 "#PWR016" H 8150 2650 50  0001 C CNN
 F 1 "GND" H 8150 2750 50  0000 C CNN
 F 2 "" H 8150 2900 50  0001 C CNN
@@
 $EndComp
 $Comp
-L GND #PWR?
+L GND #PWR017
 U 1 1 5AFEA7BF
 P 8450 2100
-F 0 "#PWR?" H 8450 1850 50  0001 C CNN
+F 0 "#PWR017" H 8450 1850 50  0001 C CNN
 F 1 "GND" H 8450 1950 50  0000 C CNN
 F 2 "" H 8450 2100 50  0001 C CNN
@@
 $EndComp
 $Comp
-L GND #PWR?
+L GND #PWR018
 U 1 1 5AFEA7DD
 P 6300 2100
-F 0 "#PWR?" H 6300 1850 50  0001 C CNN
+F 0 "#PWR018" H 6300 1850 50  0001 C CNN
 F 1 "GND" H 6300 1950 50  0000 C CNN
 F 2 "" H 6300 2100 50  0001 C CNN
@@
 	1    0    0    -1
 $EndComp
+Wire Wire Line
+	6100 2900 6650 2900
+Wire Wire Line
+	6650 2900 6650 950
+Wire Wire Line
+	6650 950  4700 950
+Wire Wire Line
+	3700 1350 3700 3700
+Wire Wire Line
+	3700 3700 8250 3700
+Wire Wire Line
+	8250 3700 8250 2900
+Wire Wire Line
+	7050 2450 7050 3550
+Connection ~ 7050 3550
+Wire Wire Line
+	5900 3550 8050 3550
+Wire Wire Line
+	8050 3550 8050 2900
+Wire Wire Line
+	5900 2900 5900 3550
+$Comp
+L GND #PWR019
+U 1 1 5AF82B3B
+P 5700 2900
+F 0 "#PWR019" H 5700 2650 50  0001 C CNN
+F 1 "GND" H 5700 2750 50  0000 C CNN
+F 2 "" H 5700 2900 50  0001 C CNN
+F 3 "" H 5700 2900 50  0001 C CNN
+	1    5700 2900
+	1    0    0    -1
+$EndComp
+$Comp
+L GND #PWR020
+U 1 1 5AF82E31
+P 7850 2900
+F 0 "#PWR020" H 7850 2650 50  0001 C CNN
+F 1 "GND" H 7850 2750 50  0000 C CNN
+F 2 "" H 7850 2900 50  0001 C CNN
+F 3 "" H 7850 2900 50  0001 C CNN
+	1    7850 2900
+	1    0    0    -1
+$EndComp
