File: hardware/gun_ir_receiver/gun_ir_receiver.sch (KiCad schematic (older format))
At the start: 3 parts

Commit message: Added led
Parts:
- LEDPL9823: footprint Connector_PinSocket_2.54mm:PinSocket_1x04_P2.54mm_Vertical -> LED_THT:LED_D5.0mm-4_RGB_Wide_Pins
Changed lines of the file:
@@
 F 0 "LEDPL9823" V 2940 812 50  0000 R CNN
 F 1 "Conn_01x04_Female" V 2849 812 50  0000 R CNN
-F 2 "Connector_PinSocket_2.54mm:PinSocket_1x04_P2.54mm_Vertical" H 3000 1100 50  0001 C CNN
+F 2 "LED_THT:LED_D5.0mm-4_RGB_Wide_Pins" H 3000 1100 50  0001 C CNN
 F 3 "~" H 3000 1100 50  0001 C CNN
 	1    3000 1100
@@
 	3750 2300 3750 2800
 $Comp
-L power:GND #PWR?
+L power:GND #PWR0105
 U 1 1 5BF5D905
 P 3550 2800
-F 0 "#PWR?" H 3550 2550 50  0001 C CNN
+F 0 "#PWR0105" H 3550 2550 50  0001 C CNN
 F 1 "GND" H 3555 2627 50  0000 C CNN
 F 2 "" H 3550 2800 50  0001 C CNN

Commit message: Added led
Parts:
- LEDPL9823: footprint LED_THT:LED_D5.0mm-4_RGB_Wide_Pins -> Connector_PinSocket_2.54mm:PinSocket_1x04_P2.54mm_Vertical
Changed lines of the file:
@@
 F 0 "LEDPL9823" V 2940 812 50  0000 R CNN
 F 1 "Conn_01x04_Female" V 2849 812 50  0000 R CNN
-F 2 "LED_THT:LED_D5.0mm-4_RGB_Wide_Pins" H 3000 1100 50  0001 C CNN
+F 2 "Connector_PinSocket_2.54mm:PinSocket_1x04_P2.54mm_Vertical" H 3000 1100 50  0001 C CNN
 F 3 "~" H 3000 1100 50  0001 C CNN
 	1    3000 1100
