File: hardware/mainboard_3.0/mainboard_3/mainboard_3.sch (KiCad schematic (older format))
At the start: 7 parts

Commit message: Start adding input connectors
Parts:
- removed J?: Conn_01x04, symbol Connector_Generic:Conn_01x04
- added ButtonConnector, MotorConnector: Conn_01x03, symbol Connector_Generic:Conn_01x03
- added DisplayConnector: Conn_01x04, symbol Connector_Generic:Conn_01x04
- added IRGunReceiverConnector: Conn_01x05, symbol Connector_Generic:Conn_01x05
- gave numbers to parts that had none: 4
Connections:
- net +3V3: now also DisplayConnector.1 (Pin_1)
- net +5V: now also IRGunReceiverConnector.4 (Pin_4), MotorConnector.3 (Pin_3)
- net GND: now also DisplayConnector.4 (Pin_4), IRGunReceiverConnector.5 (Pin_5), MotorConnector.2 (Pin_2)
- net IR_REC: now also IRGunReceiverConnector.3 (Pin_3)
- net LED_IN: now also IRReceiverConnector.1 (Pin_1), IRGunReceiverConnector.1 (Pin_1)
- net LED_OUT: now also IRGunReceiverConnector.2 (Pin_2); no longer IRReceiverConnector.1 (Pin_1)
Changed lines of the file:
@@
 $EndDescr
 $Comp
-L SparkFun-Boards:SPARKFUN_LOGIC_LEVEL_CONVERTER B?
+L SparkFun-Boards:SPARKFUN_LOGIC_LEVEL_CONVERTER LVL_Shifter
 U 1 1 5C050D11
 P 5100 3800
-F 0 "B?" H 5100 4460 45  0000 C CNN
+F 0 "LVL_Shifter" H 5100 4460 45  0000 C CNN
 F 1 "SPARKFUN_LOGIC_LEVEL_CONVERTER" H 5100 4376 45  0000 C CNN
 F 2 "SPARKFUN_LOGIC_LEVEL_CONVERTER" H 5100 4250 20  0001 C CNN
@@
 $EndComp
 $Comp
-L Connector_Generic:Conn_01x05 J?
+L Connector_Generic:Conn_01x05 IRSenderConnector
 U 1 1 5C053701
 P 7300 2900
-F 0 "J?" H 7380 2942 50  0000 L CNN
+F 0 "IRSenderConnector" H 7380 2942 50  0000 L CNN
 F 1 "Conn_01x05" H 7380 2851 50  0000 L CNN
 F 2 "" H 7300 2900 50  0001 C CNN
@@
 $EndComp
 $Comp
-L Connector_Generic:Conn_01x02 J?
+L Connector_Generic:Conn_01x02 PowerConnector
 U 1 1 5C053854
 P 3950 2400
-F 0 "J?" H 4030 2392 50  0000 L CNN
+F 0 "PowerConnector" H 4030 2392 50  0000 L CNN
 F 1 "Conn_01x02" H 4030 2301 50  0000 L CNN
 F 2 "" H 3950 2400 50  0001 C CNN
@@
 IR_GND
 $Comp
-L Connector_Generic:Conn_01x04 J?
+L Connector_Generic:Conn_01x04 IRReceiverConnector
 U 1 1 5C053B4C
 P 7500 3650
-F 0 "J?" H 7580 3642 50  0000 L CNN
+F 0 "IRReceiverConnector" H 7580 3642 50  0000 L CNN
 F 1 "Conn_01x04" H 7580 3551 50  0000 L CNN
 F 2 "" H 7500 3650 50  0001 C CNN
@@
 Wire Wire Line
 	7100 2350 7750 2350
-Wire Wire Line
-	7750 2350 7750 3350
-Wire Wire Line
-	7750 3350 7300 3350
-Wire Wire Line
-	7300 3350 7300 3550
 Text Label 7750 3100 0    50   ~ 0
 LED_OUT
 Wire Wire Line
-	5750 3600 7250 3600
+	5750 3600 6950 3600
 Wire Wire Line
 	7250 3600 7250 3650
@@
 IR_REC
 $Comp
-L Connector_Generic:Conn_01x04 J?
-U 1 1 5C0540C3
-P 5450 4750
-F 0 "J?" H 5530 4742 50  0000 L CNN
-F 1 "Conn_01x04" H 5530 4651 50  0000 L CNN
-F 2 "" H 5450 4750 50  0001 C CNN
-F 3 "~" H 5450 4750 50  0001 C CNN
-	1    5450 4750
-	1    0    0    -1
-$EndComp
-$Comp
-L power:GND #PWR?
-U 1 1 5C054126
-P 5250 4650
-F 0 "#PWR?" H 5250 4400 50  0001 C CNN
-F 1 "GND" V 5255 4522 50  0000 R CNN
-F 2 "" H 5250 4650 50  0001 C CNN
-F 3 "" H 5250 4650 50  0001 C CNN
-	1    5250 4650
-	0    1    1    0
-$EndComp
-$Comp
-L power:+5V #PWR?
-U 1 1 5C05416B
-P 5250 4750
-F 0 "#PWR?" H 5250 4600 50  0001 C CNN
-F 1 "+5V" V 5265 4878 50  0000 L CNN
-F 2 "" H 5250 4750 50  0001 C CNN
-F 3 "" H 5250 4750 50  0001 C CNN
-	1    5250 4750
-	0    -1   -1   0
+L Connector_Generic:Conn_01x03 MotorConnector
+U 1 1 5C0E9ADF
+P 6400 5250
+F 0 "MotorConnector" H 6480 5292 50  0000 L CNN
+F 1 "Conn_01x03" H 6480 5201 50  0000 L CNN
+F 2 "" H 6400 5250 50  0001 C CNN
+F 3 "~" H 6400 5250 50  0001 C CNN
+	1    6400 5250
+	1    0    0    -1
+$EndComp
+$Comp
+L power:GND #PWR?
+U 1 1 5C0E9F73
+P 7400 4600
+F 0 "#PWR?" H 7400 4350 50  0001 C CNN
+F 1 "GND" V 7405 4472 50  0000 R CNN
+F 2 "" H 7400 4600 50  0001 C CNN
+F 3 "" H 7400 4600 50  0001 C CNN
+	1    7400 4600
+	0    1    1    0
+$EndComp
+$Comp
+L power:+5V #PWR?
+U 1 1 5C0E9FF8
+P 7400 4500
+F 0 "#PWR?" H 7400 4350 50  0001 C CNN
+F 1 "+5V" V 7415 4628 50  0000 L CNN
+F 2 "" H 7400 4500 50  0001 C CNN
+F 3 "" H 7400 4500 50  0001 C CNN
+	1    7400 4500
+	0    -1   -1   0
+$EndComp
+$Comp
+L power:+5V #PWR?
+U 1 1 5C0EA54F
+P 6200 5350
+F 0 "#PWR?" H 6200 5200 50  0001 C CNN
+F 1 "+5V" V 6215 5478 50  0000 L CNN
+F 2 "" H 6200 5350 50  0001 C CNN
+F 3 "" H 6200 5350 50  0001 C CNN
+	1    6200 5350
+	0    -1   -1   0
+$EndComp
+$Comp
+L power:GND #PWR?
+U 1 1 5C0EA5B7
+P 6200 5250
+F 0 "#PWR?" H 6200 5000 50  0001 C CNN
+F 1 "GND" V 6205 5122 50  0000 R CNN
+F 2 "" H 6200 5250 50  0001 C CNN
+F 3 "" H 6200 5250 50  0001 C CNN
+	1    6200 5250
+	0    1    1    0
+$EndComp
+$Comp
+L Connector_Generic:Conn_01x05 IRGunReceiverConnector
+U 1 1 5C0EA895
+P 7600 4400
+F 0 "IRGunReceiverConnector" H 7680 4442 50  0000 L CNN
+F 1 "Conn_01x05" H 7680 4351 50  0000 L CNN
+F 2 "" H 7600 4400 50  0001 C CNN
+F 3 "~" H 7600 4400 50  0001 C CNN
+	1    7600 4400
+	1    0    0    -1
+$EndComp
+Wire Wire Line
+	7400 4400 6950 4400
+Wire Wire Line
+	6950 4400 6950 3600
+Connection ~ 6950 3600
+Wire Wire Line
+	6950 3600 7250 3600
+Wire Wire Line
+	7750 4100 7250 4100
+Wire Wire Line
+	7250 4100 7250 4300
+Wire Wire Line
+	7250 4300 7400 4300
+Wire Wire Line
+	7750 2350 7750 4100
+Wire Wire Line
+	7400 4200 7400 4000
+Wire Wire Line
+	7400 4000 8100 4000
+Wire Wire Line
+	8100 4000 8100 3300
+Wire Wire Line
+	8100 3300 7300 3300
+Wire Wire Line
+	7300 3300 7300 3550
+Text Label 8100 3500 0    50   ~ 0
+LED_IN
+$Comp
+L Connector_Generic:Conn_01x04 DisplayConnector
+U 1 1 5C0EB37F
+P 5350 1300
+F 0 "DisplayConnector" H 5430 1292 50  0000 L CNN
+F 1 "Conn_01x04" H 5430 1201 50  0000 L CNN
+F 2 "" H 5350 1300 50  0001 C CNN
+F 3 "~" H 5350 1300 50  0001 C CNN
+	1    5350 1300
+	1    0    0    -1
+$EndComp
+$Comp
+L power:GND #PWR?
+U 1 1 5C0EB403
+P 5150 1500
+F 0 "#PWR?" H 5150 1250 50  0001 C CNN
+F 1 "GND" V 5155 1372 50  0000 R CNN
+F 2 "" H 5150 1500 50  0001 C CNN
+F 3 "" H 5150 1500 50  0001 C CNN
+	1    5150 1500
+	0    1    1    0
+$EndComp
+$Comp
+L power:+3.3V #PWR?
+U 1 1 5C0EB47A
+P 5150 1200
+F 0 "#PWR?" H 5150 1050 50  0001 C CNN
+F 1 "+3.3V" V 5165 1328 50  0000 L CNN
+F 2 "" H 5150 1200 50  0001 C CNN
+F 3 "" H 5150 1200 50  0001 C CNN
+	1    5150 1200
+	0    -1   -1   0
+$EndComp
+$Comp
+L Connector_Generic:Conn_01x03 ButtonConnector
+U 1 1 5C0EB641
+P 7200 1450
+F 0 "ButtonConnector" H 7280 1492 50  0000 L CNN
+F 1 "Conn_01x03" H 7280 1401 50  0000 L CNN
+F 2 "" H 7200 1450 50  0001 C CNN
+F 3 "~" H 7200 1450 50  0001 C CNN
+	1    7200 1450
+	1    0    0    -1
 $EndComp
 $EndSCHEMATC

Commit message: More work on the pcb
Parts:
- removed PowerConnector: Conn_01x02, symbol Connector_Generic:Conn_01x02
- added Esp32Connector: Conn_01x14, symbol Connector_Generic:Conn_01x14
- added JQ6500: Conn_01x08, symbol Connector_Generic:Conn_01x08
- added PowerConnector: Screw_Terminal_01x02, symbol Connector:Screw_Terminal_01x02
- added Speaker: Conn_01x02, symbol Connector_Generic:Conn_01x02
Connections:
- net +3V3: now also Esp32Connector.2 (Pin_2)
- net +5V: now also JQ6500.5 (Pin_5), PowerConnector.2 (Pin_2)
- net GND: now also Esp32Connector.1 (Pin_1), JQ6500.6 (Pin_6), PowerConnector.1 (Pin_1)
- new net SPK+: JQ6500.1 (Pin_1), Speaker.2 (Pin_2)
- new net SPK-: JQ6500.2 (Pin_2), Speaker.1 (Pin_1)
- no-connect marks 0 -> 2
Changed lines of the file:
@@
-$EndComp
-$Comp
-L Connector_Generic:Conn_01x02 PowerConnector
-U 1 1 5C053854
-P 3950 2400
-F 0 "PowerConnector" H 4030 2392 50  0000 L CNN
-F 1 "Conn_01x02" H 4030 2301 50  0000 L CNN
-F 2 "" H 3950 2400 50  0001 C CNN
-F 3 "~" H 3950 2400 50  0001 C CNN
-	1    3950 2400
-	1    0    0    -1
 $EndComp
 $Comp
@@
 	1    0    0    -1
 $EndComp
+$Comp
+L Connector_Generic:Conn_01x08 JQ6500
+U 1 1 5C387148
+P 3800 4950
+F 0 "JQ6500" H 3880 4942 50  0000 L CNN
+F 1 "Conn_01x08" H 3880 4851 50  0000 L CNN
+F 2 "" H 3800 4950 50  0001 C CNN
+F 3 "~" H 3800 4950 50  0001 C CNN
+	1    3800 4950
+	1    0    0    -1
+$EndComp
+$Comp
+L power:GND #PWR?
+U 1 1 5C387275
+P 3600 5150
+F 0 "#PWR?" H 3600 4900 50  0001 C CNN
+F 1 "GND" V 3605 5022 50  0000 R CNN
+F 2 "" H 3600 5150 50  0001 C CNN
+F 3 "" H 3600 5150 50  0001 C CNN
+	1    3600 5150
+	0    1    1    0
+$EndComp
+$Comp
+L power:+5V #PWR?
+U 1 1 5C3872ED
+P 3600 5050
+F 0 "#PWR?" H 3600 4900 50  0001 C CNN
+F 1 "+5V" V 3615 5178 50  0000 L CNN
+F 2 "" H 3600 5050 50  0001 C CNN
+F 3 "" H 3600 5050 50  0001 C CNN
+	1    3600 5050
+	0    -1   -1   0
+$EndComp
+NoConn ~ 3600 4950
+NoConn ~ 3600 4850
+$Comp
+L Connector_Generic:Conn_01x02 Speaker
+U 1 1 5C38789C
+P 2750 4750
+F 0 "Speaker" H 2670 4425 50  0000 C CNN
+F 1 "Conn_01x02" H 2670 4516 50  0000 C CNN
+F 2 "" H 2750 4750 50  0001 C CNN
+F 3 "~" H 2750 4750 50  0001 C CNN
+	1    2750 4750
+	-1   0    0    1
+$EndComp
+Wire Wire Line
+	2950 4650 3600 4650
+Wire Wire Line
+	2950 4750 3600 4750
+Text Label 3150 4650 0    50   ~ 0
+SPK+
+Text Label 3150 4750 0    50   ~ 0
+SPK-
+$Comp
+L Connector_Generic:Conn_01x14 Esp32Connector
+U 1 1 5C389F02
+P 2850 3150
+F 0 "Esp32Connector" H 2770 2225 50  0000 C CNN
+F 1 "Conn_01x14" H 2770 2316 50  0000 C CNN
+F 2 "" H 2850 3150 50  0001 C CNN
+F 3 "~" H 2850 3150 50  0001 C CNN
+	1    2850 3150
+	-1   0    0    1
+$EndComp
+$Comp
+L Connector:Screw_Terminal_01x02 PowerConnector
+U 1 1 5C38A017
+P 3950 2400
+F 0 "PowerConnector" H 4030 2392 50  0000 L CNN
+F 1 "Screw_Terminal_01x02" H 4030 2301 50  0000 L CNN
+F 2 "" H 3950 2400 50  0001 C CNN
+F 3 "~" H 3950 2400 50  0001 C CNN
+	1    3950 2400
+	1    0    0    -1
+$EndComp
+$Comp
+L power:GND #PWR?
+U 1 1 5C38AAB0
+P 3050 3750
+F 0 "#PWR?" H 3050 3500 50  0001 C CNN
+F 1 "GND" V 3055 3622 50  0000 R CNN
+F 2 "" H 3050 3750 50  0001 C CNN
+F 3 "" H 3050 3750 50  0001 C CNN
+	1    3050 3750
+	0    -1   -1   0
+$EndComp
+$Comp
+L power:+3.3V #PWR?
+U 1 1 5C38AB27
+P 3050 3650
+F 0 "#PWR?" H 3050 3500 50  0001 C CNN
+F 1 "+3.3V" V 3065 3778 50  0000 L CNN
+F 2 "" H 3050 3650 50  0001 C CNN
+F 3 "" H 3050 3650 50  0001 C CNN
+	1    3050 3650
+	0    1    1    0
+$EndComp
 $EndSCHEMATC
